File: hardware/controlpcb/kicad-source/JECCbotESP32.sch (KiCad schematic (older format))
At the start: 15 parts, among them SW1 TAST_VER, SW2 TAST_VER, U1 ESP32_WROOM_32, U2 74xx4052, U3 74xx4052, U4 TCA9534

Commit message: added kicad source
Parts:
- added C47: 100nF, capacitors:C_0603, symbol devices:C_0603
- added R7: DNI, resistors:R_0603, symbol devices:R_0603
- added U5: ADS1015, SSOP:MSOP-10_3x3mm_Pitch0.5mm, symbol IC_interface_i2c:ADS1015
- C2, C3: value 10u -> 10uF
Connections:
- net labels added: ADC, DRIVE_BEMF1, DRIVE_BEMF2, DRIVE_INH, DRIVE_IS, DRIVE_PWM1, DRIVE_PWM2, DRIVE_PWM3, DRIVE_PWM4, GPIO5, KNIFE_INH, KNIFE_IS, KNIFE_PWM, VBAT_SENSE
- net labels removed: BAT_LVL1, BAT_LVL2, BEMF1, BEMF2, INH, IS1, IS2, KNIFE, PWM1, PWM2, PWM3, PWM4
- wire segments 149 -> 162
- no-connect marks 7 -> 10
Other:
- moved on the sheet: R5, U2, U3, U4

Commit message: changed power supply
Parts:
- U2, U3: symbol IC_logic:74xx4052 -> JECCbotESP32-rescue:74xx4052-IC_logic
Changed lines of the file:
@@
 RX
 $Comp
-L IC_logic:74xx4052 U2
+L JECCbotESP32-rescue:74xx4052-IC_logic U2
 U 1 1 5ECC1718
 P 8900 2100
@@
 MUX1_B
 $Comp
-L IC_logic:74xx4052 U3
+L JECCbotESP32-rescue:74xx4052-IC_logic U3
 U 1 1 5ED2CC29
 P 8850 3350
